File: Hardware/CoverUI/Switch.kicad_sch (KiCad schematic)
At the start: 18 parts, among them SW1 SW_MEC_5G, SW10 SW_MEC_5G, SW11 SW_MEC_5G, SW12 SW_MEC_5G, SW13 SW_MEC_5G, SW14 SW_MEC_5G, SW2 SW_MEC_5G, SW3 SW_MEC_5G, SW4 SW_MEC_5G, SW5 SW_MEC_5G, SW6 SW_MEC_5G, SW7 SW_MEC_5G, SW8 SW_MEC_5G, SW9 SW_MEC_5G

Commit message: fix(ui): update switches to 4.5mm
Parts:
- SW1, SW10, SW11, SW12, SW13, SW14, SW2, SW3, SW4, SW5, SW6, SW7, SW8, SW9: footprint lcsc:KEY-SMD_4P-L6.0-W6.0-P3.90-LS9.0 -> lcsc:SW-SMD_4P-L4.5-W4.5-P3.00-LS7.0
Changed lines of the file:
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@@
       (effects (font (size 1.27 1.27)) hide)
     )
-    (property "Footprint" "lcsc:KEY-SMD_4P-L6.0-W6.0-P3.90-LS9.0" (id 2) (at 144.78 53.34 0)
+    (property "Footprint" "lcsc:SW-SMD_4P-L4.5-W4.5-P3.00-LS7.0" (id 2) (at 144.78 53.34 0)
       (effects (font (size 1.27 1.27)) hide)
     )
@@
       (effects (font (size 1.27 1.27)) hide)
     )
-    (property "Footprint" "lcsc:KEY-SMD_4P-L6.0-W6.0-P3.90-LS9.0" (id 2) (at 120.65 36.83 0)
+    (property "Footprint" "lcsc:SW-SMD_4P-L4.5-W4.5-P3.00-LS7.0" (id 2) (at 120.65 36.83 0)
       (effects (font (size 1.27 1.27)) hide)
     )
@@
       (effects (font (size 1.27 1.27)) hide)
     )
-    (property "Footprint" "lcsc:KEY-SMD_4P-L6.0-W6.0-P3.90-LS9.0" (id 2) (at 168.91 36.83 0)
+    (property "Footprint" "lcsc:SW-SMD_4P-L4.5-W4.5-P3.00-LS7.0" (id 2) (at 168.91 36.83 0)
       (effects (font (size 1.27 1.27)) hide)
     )
@@
       (effects (font (size 1.27 1.27)) hide)
     )
-    (property "Footprint" "lcsc:KEY-SMD_4P-L6.0-W6.0-P3.90-LS9.0" (id 2) (at 193.04 69.85 0)
+    (property "Footprint" "lcsc:SW-SMD_4P-L4.5-W4.5-P3.00-LS7.0" (id 2) (at 193.04 69.85 0)
       (effects (font (size 1.27 1.27)) hide)
     )
@@
       (effects (font (size 1.27 1.27)) hide)
     )
-    (property "Footprint" "lcsc:KEY-SMD_4P-L6.0-W6.0-P3.90-LS9.0" (id 2) (at 144.78 36.83 0)
+    (property "Footprint" "lcsc:SW-SMD_4P-L4.5-W4.5-P3.00-LS7.0" (id 2) (at 144.78 36.83 0)
       (effects (font (size 1.27 1.27)) hide)
     )
@@
       (effects (font (size 1.27 1.27)) hide)
     )
-    (property "Footprint" "lcsc:KEY-SMD_4P-L6.0-W6.0-P3.90-LS9.0" (id 2) (at 120.65 53.34 0)
+    (property "Footprint" "lcsc:SW-SMD_4P-L4.5-W4.5-P3.00-LS7.0" (id 2) (at 120.65 53.34 0)
       (effects (font (size 1.27 1.27)) hide)
     )
@@
       (effects (font (size 1.27 1.27)) hide)
     )
-    (property "Footprint" "lcsc:KEY-SMD_4P-L6.0-W6.0-P3.90-LS9.0" (id 2) (at 120.65 69.85 0)
+    (property "Footprint" "lcsc:SW-SMD_4P-L4.5-W4.5-P3.00-LS7.0" (id 2) (at 120.65 69.85 0)
       (effects (font (size 1.27 1.27)) hide)
     )
@@
       (effects (font (size 1.27 1.27)) hide)
     )
-    (property "Footprint" "lcsc:KEY-SMD_4P-L6.0-W6.0-P3.90-LS9.0" (id 2) (at 120.65 87.63 0)
+    (property "Footprint" "lcsc:SW-SMD_4P-L4.5-W4.5-P3.00-LS7.0" (id 2) (at 120.65 87.63 0)
       (effects (font (size 1.27 1.27)) hide)
     )
@@
       (effects (font (size 1.27 1.27)) hide)
     )
-    (property "Footprint" "lcsc:KEY-SMD_4P-L6.0-W6.0-P3.90-LS9.0" (id 2) (at 168.91 53.34 0)
+    (property "Footprint" "lcsc:SW-SMD_4P-L4.5-W4.5-P3.00-LS7.0" (id 2) (at 168.91 53.34 0)
       (effects (font (size 1.27 1.27)) hide)
     )
@@
       (effects (font (size 1.27 1.27)) hide)
     )
-    (property "Footprint" "lcsc:KEY-SMD_4P-L6.0-W6.0-P3.90-LS9.0" (id 2) (at 144.78 87.63 0)
+    (property "Footprint" "lcsc:SW-SMD_4P-L4.5-W4.5-P3.00-LS7.0" (id 2) (at 144.78 87.63 0)
       (effects (font (size 1.27 1.27)) hide)
     )
@@
       (effects (font (size 1.27 1.27)) hide)
     )
-    (property "Footprint" "lcsc:KEY-SMD_4P-L6.0-W6.0-P3.90-LS9.0" (id 2) (at 168.91 69.85 0)
+    (property "Footprint" "lcsc:SW-SMD_4P-L4.5-W4.5-P3.00-LS7.0" (id 2) (at 168.91 69.85 0)
       (effects (font (size 1.27 1.27)) hide)
     )
@@
       (effects (font (size 1.27 1.27)) hide)
     )
-    (property "Footprint" "lcsc:KEY-SMD_4P-L6.0-W6.0-P3.90-LS9.0" (id 2) (at 193.04 36.83 0)
+    (property "Footprint" "lcsc:SW-SMD_4P-L4.5-W4.5-P3.00-LS7.0" (id 2) (at 193.04 36.83 0)
       (effects (font (size 1.27 1.27)) hide)
     )
@@
       (effects (font (size 1.27 1.27)) hide)
     )
-    (property "Footprint" "lcsc:KEY-SMD_4P-L6.0-W6.0-P3.90-LS9.0" (id 2) (at 193.04 53.34 0)
+    (property "Footprint" "lcsc:SW-SMD_4P-L4.5-W4.5-P3.00-LS7.0" (id 2) (at 193.04 53.34 0)
       (effects (font (size 1.27 1.27)) hide)
     )
@@
       (effects (font (size 1.27 1.27)) hide)
     )
-    (property "Footprint" "lcsc:KEY-SMD_4P-L6.0-W6.0-P3.90-LS9.0" (id 2) (at 144.78 69.85 0)
-      (effects (font (size 1.27 1.27)) hide)
-    )
+    (property "Footprint" "lcsc:SW-SMD_4P-L4.5-W4.5-P3.00-LS7.0" (id 2) (at 144.78 69.85 0)
+      (effects (font (size 1.27 1.27)) hide)
+    )

Commit message: fix: switch lcsc part
Parts:
- SW1, SW10, SW11, SW12, SW13, SW14, SW2, SW3, SW4, SW5, SW6, SW7, SW8, SW9: LCSC Part C2834928 -> C840835
Changed lines of the file:
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@@
       (effects (font (size 1.27 1.27)) hide)
     )
-    (property "LCSC Part" "C2834928" (id 4) (at 144.78 58.42 0)
+    (property "LCSC Part" "C840835" (id 4) (at 144.78 58.42 0)
       (effects (font (size 1.27 1.27)) hide)
     )
@@
       (effects (font (size 1.27 1.27)) hide)
     )
-    (property "LCSC Part" "C2834928" (id 4) (at 120.65 41.91 0)
+    (property "LCSC Part" "C840835" (id 4) (at 120.65 41.91 0)
       (effects (font (size 1.27 1.27)) hide)
     )
@@
       (effects (font (size 1.27 1.27)) hide)
     )
-    (property "LCSC Part" "C2834928" (id 4) (at 168.91 41.91 0)
+    (property "LCSC Part" "C840835" (id 4) (at 168.91 41.91 0)
       (effects (font (size 1.27 1.27)) hide)
     )
@@
       (effects (font (size 1.27 1.27)) hide)
     )
-    (property "LCSC Part" "C2834928" (id 4) (at 193.04 74.93 0)
+    (property "LCSC Part" "C840835" (id 4) (at 193.04 74.93 0)
       (effects (font (size 1.27 1.27)) hide)
     )
@@
       (effects (font (size 1.27 1.27)) hide)
     )
-    (property "LCSC Part" "C2834928" (id 4) (at 144.78 41.91 0)
+    (property "LCSC Part" "C840835" (id 4) (at 144.78 41.91 0)
       (effects (font (size 1.27 1.27)) hide)
     )
@@
       (effects (font (size 1.27 1.27)) hide)
     )
-    (property "LCSC Part" "C2834928" (id 4) (at 120.65 58.42 0)
+    (property "LCSC Part" "C840835" (id 4) (at 120.65 58.42 0)
       (effects (font (size 1.27 1.27)) hide)
     )
@@
       (effects (font (size 1.27 1.27)) hide)
     )
-    (property "LCSC Part" "C2834928" (id 4) (at 120.65 74.93 0)
+    (property "LCSC Part" "C840835" (id 4) (at 120.65 74.93 0)
       (effects (font (size 1.27 1.27)) hide)
     )
@@
       (effects (font (size 1.27 1.27)) hide)
     )
-    (property "LCSC Part" "C2834928" (id 4) (at 120.65 92.71 0)
+    (property "LCSC Part" "C840835" (id 4) (at 120.65 92.71 0)
       (effects (font (size 1.27 1.27)) hide)
     )
@@
       (effects (font (size 1.27 1.27)) hide)
     )
-    (property "LCSC Part" "C2834928" (id 4) (at 168.91 58.42 0)
+    (property "LCSC Part" "C840835" (id 4) (at 168.91 58.42 0)
       (effects (font (size 1.27 1.27)) hide)
     )
@@
       (effects (font (size 1.27 1.27)) hide)
     )
-    (property "LCSC Part" "C2834928" (id 4) (at 144.78 92.71 0)
+    (property "LCSC Part" "C840835" (id 4) (at 144.78 92.71 0)
       (effects (font (size 1.27 1.27)) hide)
     )
@@
       (effects (font (size 1.27 1.27)) hide)
     )
-    (property "LCSC Part" "C2834928" (id 4) (at 168.91 74.93 0)
+    (property "LCSC Part" "C840835" (id 4) (at 168.91 74.93 0)
       (effects (font (size 1.27 1.27)) hide)
     )
@@
       (effects (font (size 1.27 1.27)) hide)
     )
-    (property "LCSC Part" "C2834928" (id 4) (at 193.04 41.91 0)
+    (property "LCSC Part" "C840835" (id 4) (at 193.04 41.91 0)
       (effects (font (size 1.27 1.27)) hide)
     )
@@
       (effects (font (size 1.27 1.27)) hide)
     )
-    (property "LCSC Part" "C2834928" (id 4) (at 193.04 58.42 0)
+    (property "LCSC Part" "C840835" (id 4) (at 193.04 58.42 0)
       (effects (font (size 1.27 1.27)) hide)
     )
@@
       (effects (font (size 1.27 1.27)) hide)
     )
-    (property "LCSC Part" "C2834928" (id 4) (at 144.78 74.93 0)
-      (effects (font (size 1.27 1.27)) hide)
-    )
+    (property "LCSC Part" "C840835" (id 4) (at 144.78 74.93 0)
+      (effects (font (size 1.27 1.27)) hide)
+    )
